File: Nixie_proj.sch (KiCad schematic (older format))
At the start: 8 parts

Commit message: Fertigungsdaten erstellt
Parts:
- FID1, FID2, FID3, FID4: Reichelt (none) -> n.b.; manf# (none) -> n.b.
Changed lines of the file:
@@
 F 2 "Fiducial:Fiducial_0.75mm_Mask1.5mm" H 3650 5550 50  0001 C CNN
 F 3 "~" H 3650 5550 50  0001 C CNN
+F 4 "n.b." H 3650 5550 50  0001 C CNN "Reichelt"
+F 5 "n.b." H 3650 5550 50  0001 C CNN "manf#"
 	1    3650 5550
 	1    0    0    -1
@@
 F 2 "Fiducial:Fiducial_0.75mm_Mask1.5mm" H 4050 5550 50  0001 C CNN
 F 3 "~" H 4050 5550 50  0001 C CNN
+F 4 "n.b." H 4050 5550 50  0001 C CNN "Reichelt"
+F 5 "n.b." H 4050 5550 50  0001 C CNN "manf#"
 	1    4050 5550
 	1    0    0    -1
@@
 F 2 "Fiducial:Fiducial_0.75mm_Mask1.5mm" H 4450 5550 50  0001 C CNN
 F 3 "~" H 4450 5550 50  0001 C CNN
+F 4 "n.b." H 4450 5550 50  0001 C CNN "Reichelt"
+F 5 "n.b." H 4450 5550 50  0001 C CNN "manf#"
 	1    4450 5550
 	1    0    0    -1
@@
 F 2 "Fiducial:Fiducial_0.75mm_Mask1.5mm" H 4800 5550 50  0001 C CNN
 F 3 "~" H 4800 5550 50  0001 C CNN
+F 4 "n.b." H 4800 5550 50  0001 C CNN "Reichelt"
+F 5 "n.b." H 4800 5550 50  0001 C CNN "manf#"
 	1    4800 5550
 	1    0    0    -1
