File: nixie_mcu.sch (KiCad schematic (older format))
At the start: 51 parts, among them J1 Conn_01x06_Male, Q401 BSS138, Q403 BSS138, Q404 BSS138, SW401 SW_Push, SW402 Rechts, SW403 Mitte, SW404 Links, U1 DS3231MZ, U401 ESP-12E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

Commit message: Fertigungsdaten erstellt
Parts:
- J1: Reichelt (none) -> n.b.; manf# (none) -> n.b.
Changed lines of the file:
@@
 F 2 "Connector_PinHeader_2.54mm:PinHeader_1x06_P2.54mm_Vertical" H 11250 4300 50  0001 C CNN
 F 3 "~" H 11250 4300 50  0001 C CNN
+F 4 "n.b." H 11250 4300 50  0001 C CNN "Reichelt"
+F 5 "n.b." H 11250 4300 50  0001 C CNN "manf#"
 	1    11250 4300
 	-1   0    0    -1
