File: Nixie_proj.kicad_pcb (KiCad board)
At the start: 2 copper layers, 140 x 65 mm, 119 parts, among them J1 Conn_01x06_Male, P301 USB_OTG, Q2 BSS138, Q202 MPSA92, Q203 MPSA92, Q204 MPSA92, Q205 MPSA92, Q206 MPSA92, Q207 MPSA92, Q208 MPSA92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

Commit message: Kleinigkeiten
Parts:
- moved HV TEST 0.25 mm to (37.8, 90.0)
Routing:
- net VAA: track 318.4 -> 323.6 mm
Other:
- net class VAA added: clearance 0.5, trace_width 0.6, via_dia 0.6, via_drill 0.4
- board text added: "RX 3V3"
- board text added: "SCL 5V"
- board text added: "SDA 5V"
- board text added: "TX 3V3"
- board text removed: "RX"
- board text removed: "SCL"
- board text removed: "SDA"
- board text removed: "TX"

Commit message: wenn man einmal anfängt...
Parts:
- moved C14 0.50 mm to (71.0, 100.0)
- moved C16 0.50 mm to (74.0, 100.0)
- moved C17 0.25 mm to (136.0, 100.0)
- moved C20 0.25 mm to (139.0, 100.0)
Routing:
- net Net-(LED401-Pad4): track 32.1 -> 41.6 mm
- net +5V: track 576.5 -> 570.1 mm
- net Net-(LED402-Pad4): track 46.6 -> 47.4 mm

Commit message: mal wieder aktualisiert
Parts:
- H4: value MountingHole -> eMountingHole
- P301: value USB_OTG -> USB Buchse
- RX: value RX -> GRÜN
- TX: value TX -> ROT
